Commit message: Got nav2 working after integrating panda arm

File: sonny_description/urdf/panda_gz_amm.urdf.xacro (robot description, xacro)
@@ -1,16 +1,14 @@
-<?xml version="1.0"?>
-<robot xmlns:xacro="http://www.ros.org/wiki/xacro">
-  <!-- Macro that adds the Panda arm + its ros2_control and mounts it to any parent link -->
-  <xacro:macro name="add_panda_arm" params="parent_link base_xyz:='0 0 0' base_rpy:='0 0 0'">
+<?xml version="1.0" ?>
+<robot name="panda" xmlns:xacro="http://www.ros.org/wiki/xacro">
     <xacro:include filename="$(find moveit_resources_panda_description)/urdf/panda.urdf.xacro" />
-    <!-- Fixed joint from parent link to panda_link0 -->
-    <joint name="panda_on_${parent_link}" type="fixed">
-      <parent link="${parent_link}"/>
+    <xacro:property name="mob_base_height" value="0.18"/>
+    <!-- Fixed joint from your parent link to panda_link0 -->
+    <joint name="panda_on_base_link" type="fixed">
+      <parent link="base_link"/>
       <child  link="panda_link0"/>
-      <origin xyz="${base_xyz}" rpy="${base_rpy}"/>
+      <origin xyz="0.0 0 ${mob_base_height/2}" rpy="0 0 0"/>
     </joint>
     <gazebo>
       <plugin filename="gz_ros2_control-system" name="gz_ros2_control::GazeboSimROS2ControlPlugin">
-        <!-- <parameters>/home/reuben/moveit_ws/src/sonny_description/config/ros2_controllers.yaml</parameters> -->
         <parameters>/home/reuben/moveit_ws/src/panda_moveit_config/config/ros2_controllers.yaml</parameters>
       </plugin>
@@ -68,4 +66,3 @@
       </joint>
     </ros2_control>
-  </xacro:macro>
 </robot>

File: sonny_description/urdf/sonny_base.urdf.xacro (robot description, xacro)
@@ -9,4 +9,5 @@
   <xacro:property name="base_length" value="0.42"/>
   <xacro:property name="base_height" value="0.18"/>
+  <!-- If you updates this, update mob_base_height in panda_gz_amm.urdf.xacro too  -->
   <xacro:property name="wheel_radius" value="0.10"/>
   <xacro:property name="wheel_width"  value="0.04"/>
@@ -67,5 +68,6 @@
       </geometry>
       <material name="base_cyan">
-        <color rgba="0 1 1 1"/>
+        <!-- <color rgba="0 1 1 1"/> -->
+        <color rgba="0.2 0.2 0.2 1"/>
       </material>
     </visual>
@@ -77,8 +79,8 @@
   </link>
   <!-- Mount Panda on top of the base_link -->
-  <xacro:add_panda_arm
+  <!-- <xacro:add_panda_arm
       parent_link="base_link"
-      base_xyz="0.5 0 ${base_height/2}"
-      base_rpy="0 0 0"/>
+      base_xyz="0.0 0 ${base_height/2}"
+      base_rpy="0 0 0"/> -->
   <!-- Footprint (has inertial in original SDF) -->
   <link name="base_footprint">
@@ -161,4 +163,16 @@
     <origin xyz="${caster_xoff} 0.0 ${-(base_height/2)}" rpy="0 0 0"/>
   </joint>
+  <!-- <gazebo reference="drivewhl_l_link">
+      <mu1 value="1.0"/>
+      <mu2 value="1.0"/>
+  </gazebo>
+  <gazebo reference="drivewhl_r_link">
+      <mu1 value="1.0"/>
+      <mu2 value="1.0"/>
+  </gazebo>
+  <gazebo reference="front_caster">
+      <mu1 value="1.0"/>
+      <mu2 value="1.0"/>
+  </gazebo> -->
   <!-- =========================
        IMU link
@@ -203,5 +217,6 @@
     <child  link="lidar_link"/>
     <!-- pose relative_to="base_link">0 0 0.12 0 0 0 -->
-    <origin xyz="0 0 0.12" rpy="0 0 0"/>
+    <!-- <origin xyz="0 0 0.12" rpy="0 0 0"/> -->
+    <origin xyz="${caster_xoff} 0 0.12" rpy="0 0 0"/>
   </joint>
   <!-- =========================
@@ -286,4 +301,6 @@
             <samples>360</samples>
             <resolution>1.000000</resolution>
+            <!-- <min_angle>-1.5708</min_angle>
+            <max_angle>1.5708</max_angle>            -->
             <min_angle>0.000000</min_angle>
             <max_angle>6.280000</max_angle>
@@ -306,21 +323,26 @@
   <gazebo>
     <!-- Diff drive (gz-sim system plugin, copied from SDF) -->
-    <plugin filename="gz-sim-diff-drive-system" name="gz::sim::systems::DiffDrive">
-      <!-- wheels -->
+    <!-- <plugin filename="gz-sim-diff-drive-system" name="gz::sim::systems::DiffDrive">
       <left_joint>drivewhl_l_joint</left_joint>
       <right_joint>drivewhl_r_joint</right_joint>
-      <!-- kinematics -->
       <wheel_separation>0.4</wheel_separation>
-      <wheel_radius>${wheel_radius}</wheel_radius>
-      <!-- limits -->
-      <max_linear_acceleration>0.1</max_linear_acceleration>
-      <!-- input -->
-      <topic>/demo/cmd_vel</topic>
-      <!-- output -->
+      <wheel_radius>${wheel_radius}</wheel_radius> -->
+      <!-- <max_linear_acceleration>0.1</max_linear_acceleration> -->
+      <!-- limits: tune these -->
+      <!-- <max_linear_velocity>1.0</max_linear_velocity>
+      <min_linear_velocity>-1.0</min_linear_velocity>
+      <max_angular_velocity>1.2</max_angular_velocity>
+      <min_angular_velocity>-1.2</min_angular_velocity> -->
+      <!-- key for “easier to move”: higher accel -->
+      <!-- <max_linear_acceleration>0.8</max_linear_acceleration>
+      <min_linear_acceleration>-0.8</min_linear_acceleration>
+      <max_angular_acceleration>1.5</max_angular_acceleration>
+      <min_angular_acceleration>-1.5</min_angular_acceleration> -->
+      <!-- <topic>/demo/cmd_vel</topic>
       <odom_topic>/demo/odom</odom_topic>
       <tf_topic>/tf</tf_topic>
       <frame_id>odom</frame_id>
       <child_frame_id>base_link</child_frame_id>
-    </plugin>
+    </plugin> -->
     <!-- Joint state publisher system -->
     <plugin
